File: oled-nametag.kicad_sch (KiCad schematic)
At the start: 12 parts, among them J1 USB_C_Receptacle_USB2.0, SW1 Power, SW2 BTN1, SW3 BTN2, SW4 BTN3

Commit message: Finish first layout revision
Changed lines of the file:
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@@
 (kicad_sch (version 20230121) (generator eeschema)
   (paper "A4")
+  (junction (at 113.03 54.61) (diameter 0) (color 0 0 0 0)
+  )
   (junction (at 106.68 69.85) (diameter 0) (color 0 0 0 0)
   )
@@
     (stroke (width 0) (type default))
   )
-  (wire (pts (xy 106.68 54.61) (xy 147.32 54.61))
+  (wire (pts (xy 106.68 54.61) (xy 113.03 54.61))
     (stroke (width 0) (type default))
   )
@@
     (stroke (width 0) (type default))
   )
+  (wire (pts (xy 113.03 53.34) (xy 113.03 54.61))
+    (stroke (width 0) (type default))
+  )
   (wire (pts (xy 83.82 93.98) (xy 80.01 93.98))
+    (stroke (width 0) (type default))
+  )
+  (wire (pts (xy 113.03 54.61) (xy 147.32 54.61))
     (stroke (width 0) (type default))
   )
@@
         )
       )
+    )
+  )
+  (symbol (lib_id "power:PWR_FLAG") (at 113.03 53.34 0) (unit 1)
+    (in_bom yes) (on_board yes) (dnp no) (fields_autoplaced)
+    (property "Reference" "#FLG01" (at 113.03 51.435 0)
+      (effects (font (size 1.27 1.27)) hide)
+    )
+    (property "Value" "PWR_FLAG" (at 113.03 49.8381 0)
+      (effects (font (size 1.27 1.27)))
+    )
+    (property "Footprint" "" (at 113.03 53.34 0)
+      (effects (font (size 1.27 1.27)) hide)
+    )
+    (property "Datasheet" "~" (at 113.03 53.34 0)
+      (effects (font (size 1.27 1.27)) hide)
+    )
+    (pin "1")
+    (instances
+      (project "oled-nametag"
+        (path "/c0b8a503-1da4-4e1a-941c-dddf39a5c519"
+          (reference "#FLG01") (unit 1)
+        )
+      )

Commit message: Add power rail testpoints
Parts:
- added J2: I2C, Connector_PinHeader_2.54mm:PinHeader_1x03_P2.54mm_Vertical, symbol Connector_Generic:Conn_01x03
Connections:
- net ESP32/SCL: now also J2.2 (Pin_2)
- net ESP32/SDA: now also J2.3 (Pin_3)
- net GND: now also J2.1 (Pin_1)
Changed lines of the file:
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@@
   (junction (at 113.03 54.61) (diameter 0) (color 0 0 0 0)
   )
+  (junction (at 182.88 83.82) (diameter 0) (color 0 0 0 0)
+  )
   (junction (at 106.68 69.85) (diameter 0) (color 0 0 0 0)
   )
@@
   )
   (junction (at 113.03 59.69) (diameter 0) (color 0 0 0 0)
+  )
+  (junction (at 181.61 86.36) (diameter 0) (color 0 0 0 0)
   )
   (junction (at 106.68 72.39) (diameter 0) (color 0 0 0 0)
@@
     (stroke (width 0) (type default))
   )
+  (wire (pts (xy 191.77 76.2) (xy 191.77 86.36))
+    (stroke (width 0) (type default))
+  )
   (wire (pts (xy 116.84 119.38) (xy 116.84 110.49))
     (stroke (width 0) (type default))
@@
     (stroke (width 0) (type default))
   )
+  (wire (pts (xy 181.61 86.36) (xy 181.61 97.79))
+    (stroke (width 0) (type default))
+  )
   (wire (pts (xy 176.53 121.92) (xy 210.82 121.92))
     (stroke (width 0) (type default))
@@
     (stroke (width 0) (type default))
   )
-  (wire (pts (xy 181.61 76.2) (xy 181.61 97.79))
+  (wire (pts (xy 181.61 76.2) (xy 181.61 86.36))
     (stroke (width 0) (type default))
   )
@@
     (stroke (width 0) (type default))
   )
+  (wire (pts (xy 182.88 83.82) (xy 182.88 100.33))
+    (stroke (width 0) (type default))
+  )
   (wire (pts (xy 140.97 93.98) (xy 147.32 93.98))
     (stroke (width 0) (type default))
@@
     (stroke (width 0) (type default))
   )
+  (wire (pts (xy 186.69 76.2) (xy 186.69 77.47))
+    (stroke (width 0) (type default))
+  )
   (wire (pts (xy 146.05 82.55) (xy 179.07 82.55))
     (stroke (width 0) (type default))
@@
     (stroke (width 0) (type default))
   )
+  (wire (pts (xy 189.23 83.82) (xy 182.88 83.82))
+    (stroke (width 0) (type default))
+  )
   (wire (pts (xy 176.53 93.98) (xy 179.07 93.98))
     (stroke (width 0) (type default))
@@
     (stroke (width 0) (type default))
   )
+  (wire (pts (xy 191.77 86.36) (xy 181.61 86.36))
+    (stroke (width 0) (type default))
+  )
   (wire (pts (xy 83.82 95.25) (xy 83.82 93.98))
     (stroke (width 0) (type default))
   )
-  (wire (pts (xy 182.88 73.66) (xy 182.88 100.33))
+  (wire (pts (xy 182.88 73.66) (xy 182.88 83.82))
     (stroke (width 0) (type default))
   )
@@
   )
   (wire (pts (xy 106.68 62.23) (xy 107.95 62.23))
+    (stroke (width 0) (type default))
+  )
+  (wire (pts (xy 189.23 76.2) (xy 189.23 83.82))
     (stroke (width 0) (type default))
   )
@@
         (path "/c0b8a503-1da4-4e1a-941c-dddf39a5c519"
           (reference "#PWR059") (unit 1)
+        )
+      )
+    )
+  )
+  (symbol (lib_id "power:GND") (at 186.69 77.47 0) (unit 1)
+    (in_bom yes) (on_board yes) (dnp no) (fields_autoplaced)
+    (property "Reference" "#PWR083" (at 186.69 83.82 0)
+      (effects (font (size 1.27 1.27)) hide)
+    )
+    (property "Value" "GND" (at 186.69 81.6055 0)
+      (effects (font (size 1.27 1.27)))
+    )
+    (property "Footprint" "" (at 186.69 77.47 0)
+      (effects (font (size 1.27 1.27)) hide)
+    )
+    (property "Datasheet" "" (at 186.69 77.47 0)
+      (effects (font (size 1.27 1.27)) hide)
+    )
+    (pin "1")
+    (instances
+      (project "oled-nametag"
+        (path "/c0b8a503-1da4-4e1a-941c-dddf39a5c519"
+          (reference "#PWR083") (unit 1)
         )
       )
@@
         )
       )
+    )
+  )
+  (symbol (lib_id "Connector_Generic:Conn_01x03") (at 189.23 71.12 90) (unit 1)
+    (in_bom yes) (on_board yes) (dnp yes) (fields_autoplaced)
+    (property "Reference" "J2" (at 193.802 70.4763 90)
+      (effects (font (size 1.27 1.27)) (justify right))
+    )
+    (property "Value" "I2C" (at 193.802 72.3973 90)
+      (effects (font (size 1.27 1.27)) (justify right))
+    )
+    (property "Footprint" "Connector_PinHeader_2.54mm:PinHeader_1x03_P2.54mm_Vertical" (at 189.23 71.12 0)
+      (effects (font (size 1.27 1.27)) hide)
+    )
+    (property "Datasheet" "~" (at 189.23 71.12 0)
+      (effects (font (size 1.27 1.27)) hide)
+    )
+    (pin "1")
+    (pin "2")
+    (pin "3")
+    (instances
+      (project "oled-nametag"
+        (path "/c0b8a503-1da4-4e1a-941c-dddf39a5c519"
+          (reference "J2") (unit 1)
+        )
+      )

Commit message: Add missing LCSC partnumbers
Parts:
- SW1, SW2, SW3, SW4: LCSC (none) -> C963349
Changed lines of the file:
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@@
+      (effects (font (size 1.27 1.27)) hide)
+    )
+    (property "LCSC" "C963349" (at 123.19 128.27 0)
       (effects (font (size 1.27 1.27)) hide)
     )
@@
       (effects (font (size 1.27 1.27)) hide)
     )
+    (property "LCSC" "C963349" (at 123.19 110.49 0)
+      (effects (font (size 1.27 1.27)) hide)
+    )
     (pin "1")
     (pin "2")
@@
     )
     (property "Datasheet" "https://www.mouser.de/datasheet/2/307/en-b3u-3615.pdf" (at 132.08 45.72 0)
+      (effects (font (size 1.27 1.27)) hide)
+    )
+    (property "LCSC" "C963349" (at 137.16 45.72 90)
       (effects (font (size 1.27 1.27)) hide)
     )
@@
       (effects (font (size 1.27 1.27)) hide)
     )
+    (property "LCSC" "C963349" (at 123.19 119.38 0)
+      (effects (font (size 1.27 1.27)) hide)
+    )

Commit message: Finsh first layout iteration
Parts:
- added D5: 4148WS, Diode_SMD:D_SOD-323, symbol Device:D_Small
- added D6: BAV70, Package_TO_SOT_SMD:SOT-23, symbol BAV70_Small:BAV70_Small
- added R22 (x3): 100R, Resistor_SMD:R_0402_1005Metric, symbol Device:R_Small
Connections:
- net +BATT: now also R22.1, R22.1, R22.1
- net ESP32/~{BTN1}: now also D5.2 (A)
- net ESP32/~{BTN2}: now also SW3.1, D6.1 (A1); no longer SW3.2
- net ESP32/~{BTN3}: now also D6.2 (A2)
- net GND: no longer SW2.1, SW3.1, SW4.1
- new net: R22.2, SW4.1
- new net: R22.2, SW2.1
- new net: R22.2, SW3.2
- new net Power/PWR_ON: D5.1 (K), D6.3 (K)
Other:
- sheet ESP32 ports: added CHRG_PWM; removed none
- sheet Power ports: added ISET, PWR_ON2; removed none
- moved on the sheet: C37, J1, J2, R3, R4, R5, SW2, SW3, SW4
